Commit message: 5-15

File: xacro/depthcam.xacro (robot description, xacro)
@@ -135,6 +135,9 @@
           <horizontal_fov>${85.2*deg_to_rad}</horizontal_fov>
           <image>
-            <width>1280</width>
-            <height>720</height>
+            <!-- <width>1280</width>
+            <height>720</height> -->
+            <!-- cerbrus:修改分辨率 -->
+            <width>640</width>
+            <height>480</height>
             <format>L_INT8</format>
           </image>
@@ -150,5 +153,7 @@
         </camera>
         <always_on>1</always_on>
-        <update_rate>90</update_rate>
+        <!-- <update_rate>90</update_rate> -->
+        <!-- cerbrus:修改发送频率,太高会导致track_buffer卡住 -->
+        <update_rate>15</update_rate>
         <visualize>0</visualize>
       </sensor>
@@ -157,6 +162,8 @@
           <horizontal_fov>${85.2*deg_to_rad}</horizontal_fov>
           <image>
-            <width>1280</width>
-            <height>720</height>
+            <!-- <width>1280</width>
+            <height>720</height> -->
+            <width>640</width>
+            <height>480</height>
             <format>L_INT8</format>
           </image>
@@ -172,5 +179,6 @@
         </camera>
         <always_on>1</always_on>
-        <update_rate>90</update_rate>
+        <!-- <update_rate>90</update_rate> -->
+        <update_rate>15</update_rate>
         <visualize>0</visualize>
       </sensor>
@@ -179,6 +187,6 @@
           <horizontal_fov>${85.2*deg_to_rad}</horizontal_fov>
           <image>
-            <width>1280</width>
-            <height>720</height>
+            <width>640</width>
+            <height>480</height>
           </image>
           <clip>
@@ -217,5 +225,5 @@
         <rangeMinDepth>0.2</rangeMinDepth>
         <rangeMaxDepth>10.0</rangeMaxDepth>
-        <pointCloud>false</pointCloud>
+        <pointCloud>true</pointCloud>
         <pointCloudTopicName>depth/color/points</pointCloudTopicName>
         <pointCloudCutoff>0.25</pointCloudCutoff>
@@ -233,9 +241,9 @@
               </geometry>
           </visual>
-          <collision>
+          <!-- <collision>
               <geometry>
                   <box size="0.0078 0.130 0.0192"/>
               </geometry>
-          </collision>
+          </collision> -->
           <inertial>
               <mass value="0.0615752"/>

File: xacro/tracker.xacro (robot description, xacro)
@@ -74,5 +74,5 @@
   </xacro:macro>
   <!-- INTEL REALSENSE T265 -->
-  <xacro:macro name="realsense_T265" params="sensor_name parent_link rate *origin">
+  <xacro:macro name="realsense_T265" params="sensor_name parent_link *origin rate">
     <joint name="${sensor_name}_odom_frame_joint" type="fixed">
         <parent link="${parent_link}"/>
